File: 12S.brd (EAGLE design)
At the start: 120 x 100 mm, 170 parts, among them CN1 S16B-XH-A(LF)(SN), CN2 0428202214, CN3 S16B-XH-A(LF)(SN), CN4 0428202214, Q13 BSS84-7-F, Q14 IRL640SPBF, Q15 BMS3004, Q16 IRL640SPBF, Q17 BMS3004, U1 LTC6804IG-2PBF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

Commit message: second commit
Parts:
- removed C15: 33uF, resistor:C0603
- added C26: EEE-2AA330P, SDP:CAP_EEE_G
Connections:
- net GND: now also C26.2; no longer C15.1
- net N$37: now also C26.1; no longer C15.2
Routing:
- net N$37: track 51.2 -> 68.8 mm
- net GND: track 255.8 -> 259.4 mm, vias 15 -> 16
Other:
- board text added: "/Users/TylerMatthews/Downloads/1200px-University_of_Akron_seal.bmp"
- board text removed: "/Users/TylerMatthews/Downloads/Rhinegeist.bmp"
- board text removed: "/Users/TylerMatthews/Downloads/SpaceDustIPA.bmp"
