File: 12S.sch (EAGLE design)
At the start: 170 parts, among them CN1 S16B-XH-A(LF)(SN), CN2 0428202214, CN3 S16B-XH-A(LF)(SN), CN4 0428202214, Q13 BSS84-7-F, Q14 IRL640SPBF, Q15 BMS3004, Q16 IRL640SPBF, Q17 BMS3004, U1 LTC6804IG-2PBF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

Commit message: second commit
Parts:
- removed C15: 33uF, resistor:C-EUC0603
- added C26: EEE-2AA330P, SDP:EEE-2AA330P
Connections:
- net GND: now also C26.22; no longer C15.1
- net N$37: now also C26.11; no longer C15.2
Changed lines of the file:
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@@
 <part name="D16" library="SDP" library_urn="urn:adsk.eagle:library:7995329" deviceset="LED0603" device="" package3d_urn="urn:adsk.eagle:package:8018617/2" value="RED"/>
 <part name="D13" library="SDP" library_urn="urn:adsk.eagle:library:7995329" deviceset="LED0603" device="" package3d_urn="urn:adsk.eagle:package:8018617/2" value="RED"/>
-<part name="C15" library="resistor" library_urn="urn:adsk.eagle:library:348" deviceset="C-EU" device="C0603" package3d_urn="urn:adsk.eagle:package:23616/2" value="33uF"/>
 <part name="Y1" library="SDP" library_urn="urn:adsk.eagle:library:7995329" deviceset="FOXSDLF/080-20" device="" package3d_urn="urn:adsk.eagle:package:8018637/2" value="8MHz"/>
 <part name="Q15" library="SDP" library_urn="urn:adsk.eagle:library:7995329" deviceset="BMS3004" device="" package3d_urn="urn:adsk.eagle:package:8034825/2"/>
@@
 <part name="TP15" library="SDP" library_urn="urn:adsk.eagle:library:7995329" deviceset="TP5015" device="" package3d_urn="urn:adsk.eagle:package:8035395/2"/>
 <part name="TP16" library="SDP" library_urn="urn:adsk.eagle:library:7995329" deviceset="TP5015" device="" package3d_urn="urn:adsk.eagle:package:8035395/2"/>
+<part name="C26" library="SDP" library_urn="urn:adsk.eagle:library:7995329" deviceset="EEE-2AA330P" device="" package3d_urn="urn:adsk.eagle:package:9209242/2"/>
 </parts>
 <sheets>
@@
 <attribute name="NAME" x="199.5424" y="127.2794" size="1.778" layer="95" ratio="10" rot="SR270"/>
 </instance>
-<instance part="C15" gate="G$1" x="294.64" y="99.06" rot="R180">
-<attribute name="NAME" x="293.116" y="98.679" size="1.778" layer="95" rot="R180"/>
-<attribute name="VALUE" x="293.116" y="103.759" size="1.778" layer="96" rot="R180"/>
-</instance>
 <instance part="Y1" gate="A" x="205.74" y="149.86" rot="R90">
 <attribute name="NAME" x="203.0476" y="152.1206" size="1.778" layer="95" ratio="10" rot="SR90"/>
@@
 <instance part="TP11" gate="G$1" x="190.5" y="208.28">
 <attribute name="NAME" x="187.706" y="210.312" size="1.27" layer="95"/>
+</instance>
+<instance part="C26" gate="A" x="294.64" y="101.6" rot="R270">
+<attribute name="VALUE" x="290.3728" y="104.9782" size="1.778" layer="96" ratio="10" rot="SR270"/>
+<attribute name="NAME" x="296.7228" y="100.6094" size="1.778" layer="95" ratio="10" rot="SR270"/>
 </instance>
 </instances>
@@
 <wire x1="309.88" y1="99.06" x2="309.88" y2="83.82" width="0.1524" layer="91"/>
 <pinref part="GND10" gate="1" pin="GND"/>
-<wire x1="294.64" y1="83.82" x2="309.88" y2="83.82" width="0.1524" layer="91"/>
+<wire x1="284.48" y1="83.82" x2="294.64" y2="83.82" width="0.1524" layer="91"/>
 <junction x="309.88" y="83.82"/>
 <pinref part="U3" gate="G$1" pin="GND"/>
-<pinref part="C15" gate="G$1" pin="1"/>
-<wire x1="294.64" y1="96.52" x2="294.64" y2="83.82" width="0.1524" layer="91"/>
 <pinref part="D17" gate="A" pin="1"/>
+<wire x1="294.64" y1="83.82" x2="309.88" y2="83.82" width="0.1524" layer="91"/>
 <wire x1="284.48" y1="93.98" x2="284.48" y2="83.82" width="0.1524" layer="91"/>
-<wire x1="284.48" y1="83.82" x2="294.64" y2="83.82" width="0.1524" layer="91"/>
-<junction x="294.64" y="83.82"/>
 <pinref part="C3" gate="A" pin="22"/>
 <wire x1="325.12" y1="96.52" x2="325.12" y2="83.82" width="0.1524" layer="91"/>
@@
 <wire x1="342.9" y1="83.82" x2="342.9" y2="86.36" width="0.1524" layer="91"/>
 <junction x="325.12" y="83.82"/>
+<pinref part="C26" gate="A" pin="22"/>
+<wire x1="294.64" y1="93.98" x2="294.64" y2="83.82" width="0.1524" layer="91"/>
+<junction x="294.64" y="83.82"/>
 </segment>
 <segment>
@@
 <net name="N$37" class="0">
 <segment>
-<wire x1="294.64" y1="109.22" x2="297.18" y2="109.22" width="0.1524" layer="91"/>
 <pinref part="U3" gate="G$1" pin="VIN"/>
-<pinref part="C15" gate="G$1" pin="2"/>
-<wire x1="294.64" y1="104.14" x2="294.64" y2="109.22" width="0.1524" layer="91"/>
 <pinref part="F1" gate="A" pin="2"/>
 <wire x1="281.94" y1="109.22" x2="284.48" y2="109.22" width="0.1524" layer="91"/>
-<junction x="294.64" y="109.22"/>
 <pinref part="D17" gate="A" pin="3"/>
 <wire x1="284.48" y1="109.22" x2="294.64" y2="109.22" width="0.1524" layer="91"/>
+<wire x1="294.64" y1="109.22" x2="297.18" y2="109.22" width="0.1524" layer="91"/>
 <wire x1="284.48" y1="106.68" x2="284.48" y2="109.22" width="0.1524" layer="91"/>
 <junction x="284.48" y="109.22"/>
-</segment>
-</net>
+<pinref part="C26" gate="A" pin="11"/>
+<wire x1="294.64" y1="101.6" x2="294.64" y2="109.22" width="0.1524" layer="91"/>
+<junction x="294.64" y="109.22"/>
+</segment>
+</net>
